File: MDBT42Q breakout.kicad_pcb (KiCad board)
At the start: 2 copper layers, 22.9 x 48.3 mm, 102 parts, among them J1 25, J10 3, J11 4, J12 5, J13 6, J14 7, J15 8, J16 9, J17 10, J18 24, J19 23, J2 26, J20 22, J21 DIO, J22 CLK, J23 RST, J24 20, J25 19, J26 18, J27 17, J28 16, J29 15, J3 27, J30 14, J31 13, J32 12, J33 11, J34 GND, J35 CLK, J36 DIO, J37 NC, J38 NC, J39 GND, J4 28, J40 NC, J41 VDD, J42 CTS, J43 TXD, J44 RXD, J45 RTS, J46 GND, J5 29, J6 30, J7 31, J8 VDD, J9 2, U1 MDBT42Q, Y1 32.768kHz

Commit message: change c2 c3 capacity
Parts:
- C2, C3: value 15pF -> //pF
Changed lines of the file:
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@@
     (links 101)
     (no_connects 0)
-    (area 124.409999 81.864999 147.370001 130.225001)
+    (area 106.450001 75.405 159.535715 141.765001)
     (thickness 1.6)
     (drawings 60)
@@
       (effects (font (size 1 1) (thickness 0.15)))
     )
-    (fp_text value 15pF (at 0 1.143 270) (layer F.Fab)
+    (fp_text value //pF (at 0 1.143 270) (layer F.Fab)
       (effects (font (size 0.5 0.5) (thickness 0.1)))
     )
@@
       (effects (font (size 1 1) (thickness 0.15)))
     )
-    (fp_text value 15pF (at 0 -1.143 90) (layer F.Fab)
+    (fp_text value //pF (at 0 -1.143 90) (layer F.Fab)
       (effects (font (size 0.5 0.5) (thickness 0.1)))
     )
